Commit message: don't know why radius = 0.5 isn't ussable

File: tesseract_support/urdf/online_planning_example.xacro (robot description, xacro)
@@ -61,5 +61,6 @@
       <origin xyz="0 0 1" rpy="0 0 0"/>
       <geometry>
-        <cylinder length="2" radius="0.5"/>
+        <!-- TODO: Don't know why radius 0.5 causes runtime error-->
+        <cylinder length="2" radius="1.0"/>
       </geometry>
       <material name="estop_red"/>
@@ -68,5 +69,6 @@
       <origin xyz="0 0 0" rpy="0 0 0"/>
       <geometry>
-        <cylinder length="2" radius="0.5"/>
+        <!-- TODO: Don't know why radius 0.5 causes runtime error-->
+        <cylinder length="2" radius="1.0"/>
       </geometry>
       <material name="estop_red"/>
